File: NerMo Electronics Stack I.kicad_sch (KiCad schematic)
At the start: 12 parts, among them J2 Raspberry_Pi_Zero, J4 Address_Sel

Commit message: feat: NerMo Stack V1
Parts:
- added C1: 2.2uF, Capacitor_SMD:C_0805_2012Metric, symbol Device:C
- added C2: 0.1uF, Capacitor_SMD:C_0805_2012Metric, symbol Device:C
- added C5: 470 µF, Capacitor_SMD:CP_Elec_5x3, symbol Device:C_Polarized
- added J3: Conn_02x06_Odd_Even, Connector_PinSocket_1.27mm:PinSocket_2x06_P1.27mm_Vertical, symbol Connector_Generic:Conn_02x06_Odd_Even
- added U1: MPU-6050, Sensor_Motion:InvenSense_QFN-24_4x4mm_P0.5mm, symbol Sensor_Motion:MPU-6050
- J2: footprint Custom_Modules:Raspberry_Pi_Zero_2_W_Underside_LowProfile -> Custom_Modules:Raspberry_Pi_Zero_2_W_HDR-TH
- U2: footprint Connector_PinHeader_2.54mm:PinHeader_1x05_P2.54mm_Vertical_SMD_Pin1Left -> Connector_PinHeader_2.54mm:PinHeader_1x05_P2.54mm_Vertical
Connections:
- net +3.3V: now also J3.4 (Pin_4), U1.13 (VDD), U1.8 (VLOGIC)
- net +6V: now also C5.1, J3.11 (Pin_11), J3.5 (Pin_5), J3.7 (Pin_7), J3.9 (Pin_9)
- net GND: now also C1.2, C2.2, C5.2, J3.10 (Pin_10), J3.12 (Pin_12), J3.3 (Pin_3), J3.6 (Pin_6), J3.8 (Pin_8), U1.1 (CLKIN), U1.11 (FSYNC), U1.18 (GND), U1.9 (AD0)
- net I2C_SCL: now also J3.1 (Pin_1), U1.23 (SCL)
- net I2C_SDA: now also J3.2 (Pin_2), U1.24 (SDA)
- new net: C2.1, U1.10 (REGOUT)
- new net: C1.1, U1.20 (CPOUT)
- no-connect marks 27 -> 30
Other:
- removed sheet I2C PWM Expander
- note added: "Bulk Filtering Capacitor"
- note added: "IMU onboard MP6050 6 Axis Minimum Setup"
- note added: "https://item.szlcsc.com/3137743.html"
- note removed: "https://item.szlcsc.com/3137743.html?fromZone=l_c__%2522catalog%2522&spm=sc.cidn.xh3.zy.n&lcsc_vid=QAINBgYDElBcUFBeEgVYVlMEQlVbVABeQlJcAVcDQ1gxVlNTQVJcUFdSTlBWUzsOAxUeFF5JWBYZEEoBGA4JCwFIFA4DSA%3D%3D"
- moved on the sheet: D1, D2, D3, J2, R3, R7, R9

Commit message: feat: V0.2
Parts:
- removed C5: 470 µF, Capacitor_SMD:CP_Elec_5x3, symbol Device:C_Polarized
Other:
- note removed: "Bulk Filtering Capacitor"
- moved on the sheet: J3
