File: NerMo_PowerSupply.kicad_sch (KiCad schematic)
At the start: 23 parts, among them J20 VBAT_IN, Q1 IRF7404, SW1 SW_SPDT, U3 AMS1117-3.3, U6 INA3221

Commit message: feat: NerMo Stack V1
Parts:
- added D4: LED, LED_SMD:LED_0805_2012Metric_Pad1.15x1.40mm_HandSolder, symbol Device:LED
- added R8: 3k, Resistor_SMD:R_0805_2012Metric, symbol Device:R
Connections:
- net GND is gone; now on net BAT_GND: C10.2, C11.2, C9.2, PS1.3 (GND), PS1.4 (GND), PS2.2 (GND), PS2.3 (GND), R43.2, SW1.2 (B), U3.1 (GND), U6.17 (EP), U6.3 (GND)
- net BAT_GND: now also R8.2
- net VBAT_IN: now also D4.2 (A)
- new net: D4.1 (K), R8.1
Other:
- note added: "Internal Connection"
- note added: "Power Good VBAT"

Commit message: feat: V0.2
Parts:
- added C5: 470 µF, Capacitor_SMD:CP_Elec_5x3, symbol Device:C_Polarized
- added TP1: 5V Test Point, TestPoint:TestPoint_Pad_2.0x2.0mm, symbol Connector:TestPoint
- added TP2: 3V3 Test Point, TestPoint:TestPoint_Pad_2.0x2.0mm, symbol Connector:TestPoint
- added TP3: 6V Test Point, TestPoint:TestPoint_Pad_2.0x2.0mm, symbol Connector:TestPoint
- added TP4: VBAT Test Point, TestPoint:TestPoint_Pad_2.0x2.0mm, symbol Connector:TestPoint
- added TP5: GND Test Point, TestPoint:TestPoint_Pad_2.0x2.0mm, symbol Connector:TestPoint
Connections:
- net +3.3V: now also TP2.1
- net +5V: now also C5.1, TP1.1
- net +6V: now also TP3.1
- net BAT_GND: now also C5.2, TP5.1
- net VBAT: now also TP4.1
Other:
- note added: "Bulk Filtering Capacitor"
- note added: "Test Points"
