File: Nermo_I2CExpander.kicad_sch (KiCad schematic)
At the start: 36 parts, among them J1 PWM 5, J10 PWM 8, J11 PWM 9, J12 PWM 10, J13 PWM 11, J14 PWM 12, J15 PWM 13, J16 PWM 14, J17 PWM 15, J18 PWM 16, J3 PWM 1, J5 PWM 2, J6 PWM 3, J7 PWM 4, J8 PWM 6, J9 PWM 7, U5 PCA9685PW

Commit message: feat: NerMo Stack V1
Parts:
- removed C5: 470 µF, Capacitor_SMD:CP_Elec_5x3, symbol Device:C_Polarized
- J1, J10, J11, J12, J13, J14, J3, J5, J6, J7, J8, J9: footprint Connector_Molex:Molex_PicoBlade_53261-0371_1x03-1MP_P1.25mm_Horizontal -> Connector_JST:JST_SH_SM03B-SRSS-TB_1x03-1MP_P1.00mm_Horizontal
- J15, J16, J17, J18: footprint Connector_Molex:Molex_PicoBlade_53261-0371_1x03-1MP_P1.25mm_Horizontal -> Connector_JST:JST_SH_BM03B-SRSS-TB_1x03-1MP_P1.00mm_Vertical
Connections:
- net PWM0: now also RN1.8 (R1.2); no longer RN1.1 (R1.1)
- net PWM1: now also RN1.7 (R2.2); no longer RN1.2 (R2.1)
- net PWM10: now also RN3.6 (R3.2); no longer RN3.3 (R3.1)
- net PWM11: now also RN3.5 (R4.2); no longer RN3.4 (R4.1)
- net PWM12: now also RN4.8 (R1.2); no longer RN4.1 (R1.1)
- net PWM13: now also RN4.7 (R2.2); no longer RN4.2 (R2.1)
- net PWM14: now also RN4.6 (R3.2); no longer RN4.3 (R3.1)
- net PWM15: now also RN4.5 (R4.2); no longer RN4.4 (R4.1)
- net PWM2: now also RN1.6 (R3.2); no longer RN1.3 (R3.1)
- net PWM3: now also RN1.5 (R4.2); no longer RN1.4 (R4.1)
- net PWM4: now also RN2.8 (R1.2); no longer RN2.1 (R1.1)
- net PWM5: now also RN2.7 (R2.2); no longer RN2.2 (R2.1)
- net PWM6: now also RN2.6 (R3.2); no longer RN2.3 (R3.1)
- net PWM7: now also RN2.5 (R4.2); no longer RN2.4 (R4.1)
- net PWM8: now also RN3.8 (R1.2); no longer RN3.1 (R1.1)
- net PWM9: now also RN3.7 (R2.2); no longer RN3.2 (R2.1)
- net at J8.1 (Pin_1): now also RN2.2 (R2.1); no longer RN2.7 (R2.2)
- net at J9.1 (Pin_1): now also RN2.3 (R3.1); no longer RN2.6 (R3.2)
- net at J14.1 (Pin_1): now also RN3.4 (R4.1); no longer RN3.5 (R4.2)
- net at J11.1 (Pin_1): now also RN3.1 (R1.1); no longer RN3.8 (R1.2)
- net at J10.1 (Pin_1): now also RN2.4 (R4.1); no longer RN2.5 (R4.2)
- net at J6.1 (Pin_1): now also RN1.3 (R3.1); no longer RN1.6 (R3.2)
- net at J16.1 (Pin_1): now also RN4.2 (R2.1); no longer RN4.7 (R2.2)
- net at J7.1 (Pin_1): now also RN1.4 (R4.1); no longer RN1.5 (R4.2)
- net at J1.1 (Pin_1): now also RN2.1 (R1.1); no longer RN2.8 (R1.2)
- net at J15.1 (Pin_1): now also RN4.1 (R1.1); no longer RN4.8 (R1.2)
- net at J12.1 (Pin_1): now also RN3.2 (R2.1); no longer RN3.7 (R2.2)
- net at J17.1 (Pin_1): now also RN4.3 (R3.1); no longer RN4.6 (R3.2)
- net at J5.1 (Pin_1): now also RN1.2 (R2.1); no longer RN1.7 (R2.2)
- net at J13.1 (Pin_1): now also RN3.3 (R3.1); no longer RN3.6 (R3.2)
- net at J3.1 (Pin_1): now also RN1.1 (R1.1); no longer RN1.8 (R1.2)
- net at J18.1 (Pin_1): now also RN4.4 (R4.1); no longer RN4.5 (R4.2)
Other:
- note removed: "Bulk Filtering Capacitor"

Commit message: feat: V0.2
Parts:
- added C5: 470 µF, Capacitor_Tantalum_SMD:CP_EIA-7360-38_Kemet-E_HandSolder, symbol Device:C_Polarized
Connections:
- net GND: now also C5.2
- new net +6V: C5.1
Other:
- note added: "Bulk Filtering Capacitor"
Changed lines of the file:
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@@
 	)
 	(rectangle
+		(start 226.06 116.84)
+		(end 246.38 162.56)
+		(stroke
+			(width 0)
+			(type default)
+		)
+		(fill
+			(type none)
+		)
+	)
+	(rectangle
 		(start 20.32 19.05)
 		(end 246.38 107.95)
@@
 		)
 	)
+	(text "Bulk Filtering Capacitor"
+		(exclude_from_sim no)
+		(at 237.236 115.824 0)
+		(effects
+			(font
+				(size 1.27 1.27)
+			)
+		)
+	)
 	(text "Address Pulldown"
 		(exclude_from_sim no)
@@
 	(wire
 		(pts
+			(xy 233.68 144.78) (xy 233.68 140.97)
+		)
+		(stroke
+			(width 0)
+			(type default)
+		)
+	)
+	(wire
+		(pts
 			(xy 41.91 138.43) (xy 44.45 138.43)
 		)
@@
 	(wire
 		(pts
+			(xy 233.68 130.81) (xy 233.68 133.35)
+		)
+		(stroke
+			(width 0)
+			(type default)
+		)
+	)
+	(wire
+		(pts
 			(xy 85.09 151.13) (xy 80.01 151.13)
 		)
@@
 	)
 	(symbol
+		(lib_id "power:+3.3V")
+		(at 233.68 130.81 0)
+		(unit 1)
+		(exclude_from_sim no)
+		(in_bom yes)
+		(on_board yes)
+		(dnp no)
+		(fields_autoplaced yes)
+		(property "Reference" "#PWR011"
+			(at 233.68 134.62 0)
+			(effects
+				(font
+					(size 1.27 1.27)
+				)
+				(hide yes)
+			)
+		)
+		(property "Value" "+6V"
+			(at 233.68 125.73 0)
+			(effects
+				(font
+					(size 1.27 1.27)
+				)
+			)
+		)
+		(property "Footprint" ""
+			(at 233.68 130.81 0)
+			(effects
+				(font
+					(size 1.27 1.27)
+				)
+				(hide yes)
+			)
+		)
+		(property "Datasheet" ""
+			(at 233.68 130.81 0)
+			(effects
+				(font
+					(size 1.27 1.27)
+				)
+				(hide yes)
+			)
+		)
+		(property "Description" "Power symbol creates a global label with name \"+3.3V\""
+			(at 233.68 130.81 0)
+			(effects
+				(font
+					(size 1.27 1.27)
+				)
+				(hide yes)
+			)
+		)
+		(pin "1"
+		)
+		(instances
+			(project "NerMo Electronics Stack II"
+				(path "/39dca41c-80f9-47b6-a9d6-5e39413b947c/a51c9709-1454-48ce-8eb3-8ae443d05ad0"
+					(reference "#PWR011")
+					(unit 1)
+				)
+			)
+		)
+	)
+	(symbol
 		(lib_id "Device:R")
 		(at 149.86 130.81 270)
@@
 	(symbol
 		(lib_id "power:GND")
+		(at 233.68 144.78 0)
+		(unit 1)
+		(exclude_from_sim no)
+		(in_bom yes)
+		(on_board yes)
+		(dnp no)
+		(fields_autoplaced yes)
+		(property "Reference" "#PWR055"
+			(at 233.68 151.13 0)
+			(effects
+				(font
+					(size 1.27 1.27)
+				)
+				(hide yes)
+			)
+		)
+		(property "Value" "GND"
+			(at 233.68 149.86 0)
+			(effects
+				(font
+					(size 1.27 1.27)
+				)
+			)
+		)
+		(property "Footprint" ""
+			(at 233.68 144.78 0)
+			(effects
+				(font
+					(size 1.27 1.27)
+				)
+				(hide yes)
+			)
+		)
+		(property "Datasheet" ""
+			(at 233.68 144.78 0)
+			(effects
+				(font
+					(size 1.27 1.27)
+				)
+				(hide yes)
+			)
+		)
+		(property "Description" "Power symbol creates a global label with name \"GND\" , ground"
+			(at 233.68 144.78 0)
+			(effects
+				(font
+					(size 1.27 1.27)
+				)
+				(hide yes)
+			)
+		)
+		(pin "1"
+		)
+		(instances
+			(project "NerMo Electronics Stack II"
+				(path "/39dca41c-80f9-47b6-a9d6-5e39413b947c/a51c9709-1454-48ce-8eb3-8ae443d05ad0"
+					(reference "#PWR055")
+					(unit 1)
+				)
+			)
+		)
+	)
+	(symbol
+		(lib_id "power:GND")
 		(at 54.61 36.83 0)
 		(unit 1)
@@
 					(unit 1)
 				)
+			)
+		)
+	)
+	(symbol
+		(lib_id "Device:C_Polarized")
+		(at 233.68 137.16 0)
+		(unit 1)
+		(exclude_from_sim no)
+		(in_bom yes)
+		(on_board yes)
+		(dnp no)
+		(fields_autoplaced yes)
+		(property "Reference" "C5"
+			(at 237.49 135.0009 0)
+			(effects
+				(font
+					(size 1.27 1.27)
+				)
+				(justify left)
+			)
+		)
+		(property "Value" "470 µF"
+			(at 237.49 137.5409 0)
+			(effects
+				(font
+					(size 1.27 1.27)
+				)
+				(justify left)
+			)
+		)
+		(property "Footprint" "Capacitor_Tantalum_SMD:CP_EIA-7360-38_Kemet-E_HandSolder"
+			(at 234.6452 140.97 0)
+			(effects
+				(font
+					(size 1.27 1.27)
+				)
+				(hide yes)
+			)
+		)
+		(property "Datasheet" "~"
+			(at 233.68 137.16 0)
+			(effects
+				(font
+					(size 1.27 1.27)
+				)
+				(hide yes)
+			)
+		)
+		(property "Description" "Polarized capacitor"
+			(at 233.68 137.16 0)
+			(effects
+				(font
+					(size 1.27 1.27)
+				)
+				(hide yes)
+			)
+		)
+		(pin "2"
+		)
+		(pin "1"
+		)
+		(instances
+			(project "NerMo Electronics Stack II"
+				(path "/39dca41c-80f9-47b6-a9d6-5e39413b947c/a51c9709-1454-48ce-8eb3-8ae443d05ad0"
+					(reference "C5")
+					(unit 1)
+				)
